File: stm32_pcbv1.0/stm32f103/stm32f103.kicad_pcb (KiCad board)
At the start: 2 copper layers, 86 x 45 mm, 60 parts, among them J1 SWD, J2 USART1, J3 USB1130-15-A_REVA, J4 Conn_01x30, J9 USB4105-GF-A, Q1 Q_PNP_BEC, SW1 KEY_RST, U1 LM1117-3.3, U2 STM32F103RCTx, U3 INA226AIDGSR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

Commit message: fix pcb router
Parts:
- removed J9: USB4105-GF-A, DL_Usb_TypeC_Recepatcle_SMD:DL_Usb_TypeC_Recepatcle_SMD
- removed REF** (x4): Mounting_Holes_3mm_THT, Zhbi_Mounting_Holes:Mounting_Holes_3mm_THT
- added J5: INA226 ALERT, Connector_PinSocket_2.54mm:PinSocket_1x01_P2.54mm_Vertical, F.Cu at (185.7, 104.2)
- added J6: USB1130-15-A_REVA, DL_Usb_A_USB1130-15-A_REVA:DL_Usb_A_USB1130-15-A_REVA, F.Cu at (192.1, 98.8)
- added M1: Mounting_Holes_3mm_THT, Zhbi_Mounting_Holes:Mounting_Holes_3mm_THT, F.Cu at (118.8, 79.3)
- added M2: Mounting_Holes_3mm_THT, Zhbi_Mounting_Holes:Mounting_Holes_3mm_THT, F.Cu at (196.3, 79.3)
- added M3: Mounting_Holes_3mm_THT, Zhbi_Mounting_Holes:Mounting_Holes_3mm_THT, F.Cu at (196.5, 116.0)
- added M4: Mounting_Holes_3mm_THT, Zhbi_Mounting_Holes:Mounting_Holes_3mm_THT, F.Cu at (118.7, 116.2)
- J3: value USB1130-15-A_REVA -> USB4105-GF-A; footprint DL_Usb_TypeA_Receptacle_THT:DL_Usb_TypeA_Receptacle_THT -> DL_Usb_C_USB4105-GF-A:DL_Usb_C_USB4105-GF-A
- R15: footprint Resistor_SMD:R_0805_2012Metric -> Resistor_SMD:R_2010_5025Metric
- R16, R17, R18, R19: value 10K -> 5.1K
- R23: value 220R -> 100R
- S1, S2, S3, S4: footprint DL_Button_Switch_Horizontal_THT:DL_Button_Switch_Horizontal_THT -> DL_Key_Hori_B3F-3100:DL_Key_Hori_B3F-3100
- SW1: value KEY_RST -> 1825910-6; footprint Button_Switch_SMD:SW_Push_1P1T_NO_6x6mm_H9.5mm -> DL_Key_Vertical_B3F-1000:DL_Key_Vertical_B3F-1000
- U3: footprint DL_Ina226aidgsr_Power_SMD:DL_Ina226aidgsr_Power_SMD -> DL_Ina226_INA226AIDGSR:DL_Ina226_SOP50P490X110-10N
- U4: footprint Package_SO:SOIC-8_5.23x5.23mm_P1.27mm -> DL_W25q32_W25Q32JVSSIQ:DL_W25q32_SOIC127P790X216-8N
- moved J3 76.2 mm to (116.0, 98.1), turned to 270 degrees
- moved C7 28.7 mm to (168.3, 106.4), turned to 180 degrees
- moved C6 22.3 mm to (165.7, 93.0), turned to 0 degrees
- moved R22 22.0 mm to (164.7, 106.4)
- moved C9 20.4 mm to (154.7, 108.2), turned to 180 degrees
- moved Q1 15.3 mm to (173.3, 105.1), turned to 90 degrees
- moved R23 12.7 mm to (173.3, 102.2), turned to 0 degrees
- moved R14 11.1 mm to (169.3, 103.4), turned to 0 degrees
- moved C12 5.57 mm to (136.5, 116.8)
- moved C8 4.69 mm to (151.9, 91.2)
- moved R24 4.12 mm to (164.9, 116.2), turned to 270 degrees
- moved R15 3.61 mm to (189.2, 109.6), turned to 0 degrees
- moved C10 3.51 mm to (185.1, 116.5)
- moved R6 2.94 mm to (161.9, 116.2)
- moved R10 2.71 mm to (157.5, 87.0), turned to 90 degrees
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Connections:
- J4 pad 11: /LCD_DB0 -> Net-(J4-Pad11)
- J4 pad 12: /LCD_DB1 -> Net-(J4-Pad12)
- J4 pad 13: /LCD_DB2 -> /LCD_DB7
- J4 pad 14: /LCD_DB3 -> /LCD_DB6
- J4 pad 15: /LCD_DB4 -> /LCD_DB5
- J4 pad 16: /LCD_DB5 -> /LCD_DB4
- J4 pad 17: /LCD_DB6 -> /LCD_DB3
- J4 pad 18: /LCD_DB7 -> /LCD_DB2
- J4 pad 19: Net-(J4-Pad19) -> /LCD_DB1
- J4 pad 2: +3V3 -> Net-(J4-Pad2)
- J4 pad 20: Net-(J4-Pad20) -> /LCD_DB0
- J4 pad 21: GND -> Net-(J4-Pad21)
- J4 pad 22: GND -> /LCD_RD
- J4 pad 23: GND -> /LCD_WR
- J4 pad 24: GND -> /LCD_DC
- J4 pad 25: Net-(J4-Pad25) -> /LCD_CS
- J4 pad 26: Net-(J4-Pad26) -> /LCD_RESET
- J4 pad 27: Net-(J4-Pad27) -> GND
- J4 pad 28: Net-(J4-Pad28) -> GND
- J4 pad 29: Net-(J4-Pad29) -> +3V3
- J4 pad 3: GND -> Net-(J4-Pad3)
- J4 pad 4: GND -> Net-(J4-Pad4)
- J4 pad 5: /LCD_RESET -> Net-(J4-Pad5)
- J4 pad 6: /LCD_CS -> GND
- J4 pad 7: /LCD_DC -> GND
- J4 pad 8: /LCD_WR -> GND
- J4 pad 9: /LCD_RD -> GND
- R14 pad 1: Net-(J4-Pad20) -> /BL_PWM
- R14 pad 2: Net-(Q1-Pad3) -> Net-(Q1-Pad1)
- R20 pad 1: Net-(J9-PadA5) -> Net-(J3-PadA5)
- R21 pad 2: Net-(J9-PadB5) -> Net-(J3-PadB5)
- R22 pad 2: +3V3 -> GND
- R23 pad 1: Net-(Q1-Pad1) -> Net-(Q1-Pad3)
- R23 pad 2: /BL_PWM -> Net-(J4-Pad11)
- SW1 pad 1: GND -> /RST
- U2 pad 10: /KEY3 -> Net-(U2-Pad10)
- U2 pad 11: /KEY4 -> Net-(U2-Pad11)
- U2 pad 14: /LED1 -> Net-(U2-Pad14)
- U2 pad 15: /LED2 -> /LED1
- U2 pad 16: Net-(U2-Pad16) -> /LED2
- U2 pad 2: Net-(U2-Pad2) -> /KEY2
- U2 pad 20: /LCD_CS -> Net-(U2-Pad20)
- U2 pad 21: /LCD_DC -> /SPI2_NSS
- U2 pad 22: /LCD_RESET -> /SPI2_MISO
- U2 pad 23: /LCD_WR -> /INA226_SCL
- U2 pad 24: Net-(U2-Pad24) -> /INA226_SDA
- U2 pad 25: Net-(U2-Pad25) -> /SPI2_SCLK
- U2 pad 26: /LCD_DB0 -> /SPI2_MOSI
- U2 pad 27: /LCD_DB1 -> Net-(U2-Pad27)
- U2 pad 28: /LCD_DB2 -> Net-(R22-Pad1)
- U2 pad 29: /INA226_SCL -> Net-(U2-Pad29)
- U2 pad 3: Net-(U2-Pad3) -> /KEY1
- U2 pad 30: /INA226_SDA -> Net-(U2-Pad30)
- U2 pad 33: /SPI2_NSS -> /BL_PWM
- U2 pad 34: /SPI2_SCLK -> /LCD_DB7
- U2 pad 35: /SPI2_MISO -> /LCD_DB6
- U2 pad 36: /SPI2_MOSI -> /LCD_DB5
- U2 pad 37: Net-(U2-Pad37) -> /LCD_DB4
- U2 pad 38: Net-(U2-Pad38) -> /LCD_DB3
- U2 pad 39: Net-(U2-Pad39) -> /LCD_DB2
- U2 pad 40: Net-(U2-Pad40) -> /LCD_DB1
- U2 pad 41: /LCD_RD -> /LCD_DB0
- U2 pad 50: /BL_PWM -> Net-(U2-Pad50)
- U2 pad 51: Net-(U2-Pad51) -> /LCD_RD
- U2 pad 52: Net-(U2-Pad52) -> /LCD_WR
- U2 pad 53: Net-(U2-Pad53) -> /LCD_DC
- U2 pad 54: Net-(U2-Pad54) -> /LCD_CS
- U2 pad 55: /LCD_DB3 -> Net-(U2-Pad55)
- U2 pad 56: /LCD_DB4 -> Net-(U2-Pad56)
- U2 pad 57: /LCD_DB5 -> /LCD_RESET
- U2 pad 58: /LCD_DB6 -> /KEY4
- U2 pad 59: /LCD_DB7 -> /KEY3
- U2 pad 8: /KEY1 -> Net-(U2-Pad8)
- U2 pad 9: /KEY2 -> Net-(U2-Pad9)
- U3 pad 3: Net-(R22-Pad1) -> Net-(J5-Pad1)
- U3 pad 8: +5V -> /VOUT
- U4 pad 3: Net-(U4-Pad3) -> +3V3
- U4 pad 7: Net-(U4-Pad7) -> +3V3
Routing:
- net +5V: track 111.3 -> 217.8 mm, vias 2 -> 5
- net GND: track 76.1 -> 55.6 mm, vias 36 -> 28
- net +3V3: track 251.9 -> 232.2 mm
- net /USART1_RX: track 50.1 -> 31.9 mm, vias 1 -> 2
- net /LCD_DB7: track 26.4 -> 13.7 mm
- net /VOUT: track 12.4 -> 24.6 mm, vias 0 -> 1
- net /LCD_DB6: track 25.7 -> 13.7 mm
- net /LCD_DB5: track 24.9 -> 13.7 mm
- net /KEY4: track 28.4 -> 17.3 mm, vias 2 -> 0
- net Net-(J5-Pad1): track 0.00 -> 10.6 mm
- net /LCD_DB4: track 24.2 -> 13.7 mm
- net /KEY3: track 26.8 -> 16.6 mm, vias 2 -> 0
- net /KEY2: track 28.7 -> 18.6 mm
- net /LCD_DB0: track 23.5 -> 13.7 mm
- net /LCD_DB3: track 23.4 -> 13.7 mm
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