File: stm32_pcbv1.0/stm32f103/stm32f103.sch (KiCad schematic (older format))
At the start: 56 parts, among them J1 SWD, J2 USART1, J3 USB1130-15-A_REVA, J4 Conn_01x30, J9 USB4105-GF-A, Q1 Q_PNP_BEC, SW1 KEY_RST, U1 LM1117-3.3, U2 STM32F103RCTx, U3 INA226AIDGSR, U4 W25Q32JVSS, Y1 8M

Commit message: fix pcb router
Parts:
- removed J3: USB1130-15-A_REVA, DL_Usb_TypeA_Receptacle_THT:DL_Usb_TypeA_Receptacle_THT, symbol DL_Usb_TypeA_Receptacle_THT:USB1130-15-A_REVA
- removed J9: USB4105-GF-A, DL_Usb_TypeC_Recepatcle_SMD:DL_Usb_TypeC_Recepatcle_SMD, symbol DL_Usb_TypeC_Recepatcle_SMD:USB4105-GF-A
- removed S1, S2, S3, S4: 1-1825027-1, DL_Button_Switch_Horizontal_THT:DL_Button_Switch_Horizontal_THT, symbol DL_Button_Switch_Horizontal_THT:1-1825027-1
- removed SW1: KEY_RST, Button_Switch_SMD:SW_Push_1P1T_NO_6x6mm_H9.5mm, symbol Switch:SW_Push
- removed U3: INA226AIDGSR, DL_Ina226aidgsr_Power_SMD:DL_Ina226aidgsr_Power_SMD, symbol DL_Ina226aidgsr_Power_SMD:INA226AIDGSR
- added J3: USB4105-GF-A, DL_Usb_C_USB4105-GF-A:DL_Usb_C_USB4105-GF-A, symbol DL_Usb_C_USB4105-GF-A:USB4105-GF-A
- added J5: INA226 ALERT, Connector_PinSocket_2.54mm:PinSocket_1x01_P2.54mm_Vertical, symbol Connector:Conn_01x01_Male
- added J6: USB1130-15-A_REVA, DL_Usb_A_USB1130-15-A_REVA:DL_Usb_A_USB1130-15-A_REVA, symbol DL_Usb_A_USB1130-15-A_REVA:USB1130-15-A_REVA
- added S1, S2, S3, S4: 1-1825027-1, DL_Key_Hori_B3F-3100:DL_Key_Hori_B3F-3100, symbol DL_Key_Hori_B3F-3100:1-1825027-1
- added SW1: 1825910-6, DL_Key_Vertical_B3F-1000:DL_Key_Vertical_B3F-1000, symbol DL_Key_Vertical_B3F-1000:1825910-6
- added U3: INA226AIDGSR, DL_Ina226_INA226AIDGSR:DL_Ina226_SOP50P490X110-10N, symbol DL_Ina226_INA226AIDGSR:INA226AIDGSR
- R15: footprint Resistor_SMD:R_0805_2012Metric -> Resistor_SMD:R_2010_5025Metric
- R16, R17, R18, R19: value 10K -> 5.1K
- R23: value 220R -> 100R
- U4: footprint Package_SO:SOIC-8_5.23x5.23mm_P1.27mm -> DL_W25q32_W25Q32JVSSIQ:DL_W25q32_SOIC127P790X216-8N
Connections:
- net +3V3: now also J4.29 (Pin_29), U4.3 (IO2), U4.7 (IO3), U3.6 (VS); no longer J4.2 (Pin_2), R22.2
- net +5V: now also J3.A4_B9 (VBUS), J3.B4_A9 (VBUS), U3.10 (IN+)
- net BL_PWM: now also R14.1, U2.33 (PB12); no longer R23.2, U2.50 (PA15)
- net GND: now also J4.27 (Pin_27), J4.28 (Pin_28), J4.6 (Pin_6), J4.7 (Pin_7), J4.8 (Pin_8), J4.9 (Pin_9), R22.2, J3.A1_B12 (GND), J3.B1_A12 (GND), J3.S1 (SHELL_GND), J3.S2 (SHELL_GND), J3.S3 (SHELL_GND), J3.S4 (SHELL_GND), J6.4 (GND), J6.S1 (SHIELD), J6.S2 (SHIELD), S1.1, S1.S1 (SHIELD), S1.S2 (SHIELD), S2.1, S2.S1 (SHIELD), S2.S2 (SHIELD), S3.1, S3.S1 (SHIELD), S3.S2 (SHIELD), S4.1, S4.S1 (SHIELD), S4.S2 (SHIELD), SW1.3, SW1.4, U3.7 (GND); no longer J4.21 (Pin_21), J4.22 (Pin_22), J4.23 (Pin_23), J4.24 (Pin_24), J4.3 (Pin_3), J4.4 (Pin_4)
- net INA226_SCL: now also U2.23 (PA7), U3.5 (SCL); no longer U2.29 (PB10)
- net INA226_SDA: now also U2.24 (PC4), U3.4 (SDA); no longer U2.30 (PB11)
- net KEY1: now also U2.3 (PC14); no longer U2.8 (PC0)
- net KEY2: now also U2.2 (PC13); no longer U2.9 (PC1)
- net KEY3: now also U2.59 (PB7); no longer U2.10 (PC2)
- net KEY4: now also U2.58 (PB6); no longer U2.11 (PC3)
- net LCD_CS: now also J4.25 (Pin_25), U2.54 (PD2); no longer J4.6 (Pin_6), U2.20 (PA4)
- net LCD_DB0: now also J4.20 (Pin_20), U2.41 (PA8); no longer J4.11 (Pin_11), U2.26 (PB0)
- net LCD_DB1: now also J4.19 (Pin_19), U2.40 (PC9); no longer J4.12 (Pin_12), U2.27 (PB1)
- net LCD_DB2: now also J4.18 (Pin_18), U2.39 (PC8); no longer J4.13 (Pin_13), U2.28 (PB2)
- net LCD_DB3: now also J4.17 (Pin_17), U2.38 (PC7); no longer J4.14 (Pin_14), U2.55 (PB3)
- net LCD_DB4: now also J4.16 (Pin_16), U2.37 (PC6); no longer J4.15 (Pin_15), U2.56 (PB4)
- net LCD_DB5: now also J4.15 (Pin_15), U2.36 (PB15); no longer J4.16 (Pin_16), U2.57 (PB5)
- net LCD_DB6: now also J4.14 (Pin_14), U2.35 (PB14); no longer J4.17 (Pin_17), U2.58 (PB6)
- net LCD_DB7: now also J4.13 (Pin_13), U2.34 (PB13); no longer J4.18 (Pin_18), U2.59 (PB7)
- net LCD_DC: now also J4.24 (Pin_24), U2.53 (PC12); no longer J4.7 (Pin_7), U2.21 (PA5)
- net LCD_RD: now also J4.22 (Pin_22), U2.51 (PC10); no longer J4.9 (Pin_9), U2.41 (PA8)
- net LCD_RESET: now also J4.26 (Pin_26), U2.57 (PB5); no longer J4.5 (Pin_5), U2.22 (PA6)
- net LCD_WR: now also J4.23 (Pin_23), U2.52 (PC11); no longer J4.8 (Pin_8), U2.23 (PA7)
- net LED1: now also U2.15 (PA1); no longer U2.14 (PA0)
- net LED2: now also U2.16 (PA2); no longer U2.15 (PA1)
- net RST: now also SW1.1, SW1.2
- net SPI2_MISO: now also U2.22 (PA6); no longer U2.35 (PB14)
- net SPI2_MOSI: now also U2.26 (PB0); no longer U2.36 (PB15)
- net SPI2_NSS: now also U2.21 (PA5); no longer U2.33 (PB12)
- net SPI2_SCLK: now also U2.25 (PC5); no longer U2.34 (PB13)
- net USBDN1: now also J3.A7 (DN1), J3.B7 (DN2)
- net USBDP1: now also J3.A6 (DP1), J3.B6 (DP2)
- net VOUT: now also J6.1 (VCC), U3.8 (VBUS), U3.9 (IN-)
- net at R23.1: now also Q1.3 (C); no longer Q1.1 (B)
- net at R14.2: now also Q1.1 (B); no longer Q1.3 (C)
- net at R1.1: now also S1.2
- net at R21.2: now also J3.B5 (CC2)
- net at R20.1: now also J3.A5 (CC1)
- net at R2.1: now also S2.2
- net at R3.1: now also S3.2
- net at R4.1: now also S4.2
- net at R22.1: now also U2.28 (PB2)
- net at R19.2: now also U3.1 (A1)
- net at R18.2: now also U3.2 (A0)
- new net: J5.1 (Pin_1), U3.3 (ALERT)
- new net: J4.11 (Pin_11), R23.2
- no-connect marks 29 -> 14
