File: hardware/kicad_project/stm32f103.kicad_sch (KiCad schematic)
At the start: 57 parts

Commit message: 更新 PCB 工程设置
Parts:
- J3: renamed from ?; footprint DL_Usb_C_USB4105-GF-A:DL_Usb_C_USB4105-GF-A -> 3rd_USB4105-GF-A:3rd_USB4105-GF-A(USB-C)
- J6: renamed from ?; footprint DL_Usb_A_USB1130-15-A_REVA:DL_Usb_A_USB1130-15-A_REVA -> 3rd_USB1130-15-A_REVA:3rd_USB1130-15-A_REVA(USB-A)
- S1, S2, S3, S4: renamed from ?; footprint DL_Key_Hori_B3F-3100:DL_Key_Hori_B3F-3100 -> 3rd_B3F-3100:3rd_B3F-3100(Key_Hori)
- SW1: renamed from ?; footprint DL_Key_Vertical_B3F-1000:DL_Key_Vertical_B3F-1000 -> 3rd_B3F-1000:3rd_B3F-1000(Key_Vertical)
- U3: renamed from ?; footprint DL_Ina226_INA226AIDGSR:DL_Ina226_SOP50P490X110-10N -> 3rd_INA226AIDGSR:3rd_SOP50P490X110-10N(INA226AIDGSR)
- U4: renamed from ?; footprint DL_W25q32_W25Q32JVSSIQ:DL_W25q32_SOIC127P790X216-8N -> 3rd_W25Q32JVSSIQ:3rd_SOIC127P790X216-8N(W25Q32JVSSIQ)
- gave numbers to parts that had none: 48

Commit message: 修改 PCB 库文件
Parts:
- J3: symbol DL_Usb_C_USB4105-GF-A:USB4105-GF-A -> 3rd_USB4105-GF-A(USB-C):USB4105-GF-A
- J6: symbol DL_Usb_A_USB1130-15-A_REVA:USB1130-15-A_REVA -> 3rd_USB1130-15-A_REVA(USB-A):USB1130-15-A_REVA
- S1, S2, S3, S4: symbol DL_Key_Hori_B3F-3100:1-1825027-1 -> 3rd_B3F-3100(key_Hori):1-1825027-1
- SW1: symbol DL_Key_Vertical_B3F-1000:1825910-6 -> 3rd_B3F-1000(Key_Vertical):1825910-6
- U3: symbol DL_Ina226_INA226AIDGSR:INA226AIDGSR -> 3rd_INA226AIDGSR:INA226AIDGSR
Changed lines of the file:
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@@
     (pin "1")
   )
-  (symbol (lib_id "DL_Ina226_INA226AIDGSR:INA226AIDGSR") (at 243.84 38.1 0) (unit 1)
+  (symbol (lib_id "3rd_INA226AIDGSR:INA226AIDGSR") (at 243.84 38.1 0) (unit 1)
     (in_bom yes) (on_board yes)
     (property "Reference" "U3" (id 0) (at 243.84 16.002 0))
@@
     (pin "1")
   )
-  (symbol (lib_id "DL_Usb_C_USB4105-GF-A:USB4105-GF-A") (at 243.84 81.28 0) (unit 1)
+  (symbol (lib_id "3rd_USB4105-GF-A(USB-C):USB4105-GF-A") (at 243.84 81.28 0) (unit 1)
     (in_bom yes) (on_board yes)
     (property "Reference" "J3" (id 0) (at 243.84 64.3382 0))
@@
     (pin "1")
   )
-  (symbol (lib_id "DL_Usb_A_USB1130-15-A_REVA:USB1130-15-A_REVA") (at 246.38 127 90) (unit 1)
+  (symbol (lib_id "3rd_USB1130-15-A_REVA(USB-A):USB1130-15-A_REVA") (at 246.38 127 90) (unit 1)
     (in_bom yes) (on_board yes)
     (property "Reference" "J6" (id 0) (at 257.302 128.5494 90)
@@
     (pin "1")
   )
-  (symbol (lib_id "DL_Key_Hori_B3F-3100:1-1825027-1") (at 20.32 165.1 90) (unit 1)
+  (symbol (lib_id "3rd_B3F-3100(key_Hori):1-1825027-1") (at 20.32 165.1 90) (unit 1)
     (in_bom yes) (on_board yes)
     (property "Reference" "S1" (id 0) (at 26.162 163.9316 90)
@@
     (pin "S2")
   )
-  (symbol (lib_id "DL_Key_Hori_B3F-3100:1-1825027-1") (at 35.56 165.1 90) (unit 1)
+  (symbol (lib_id "3rd_B3F-3100(key_Hori):1-1825027-1") (at 35.56 165.1 90) (unit 1)
     (in_bom yes) (on_board yes)
     (property "Reference" "S2" (id 0) (at 41.402 163.9316 90)
@@
     (pin "S2")
   )
-  (symbol (lib_id "DL_Key_Hori_B3F-3100:1-1825027-1") (at 49.53 165.1 90) (unit 1)
+  (symbol (lib_id "3rd_B3F-3100(key_Hori):1-1825027-1") (at 49.53 165.1 90) (unit 1)
     (in_bom yes) (on_board yes)
     (property "Reference" "S3" (id 0) (at 55.372 163.9316 90)
@@
     (pin "S2")
   )
-  (symbol (lib_id "DL_Key_Hori_B3F-3100:1-1825027-1") (at 63.5 165.1 90) (unit 1)
+  (symbol (lib_id "3rd_B3F-3100(key_Hori):1-1825027-1") (at 63.5 165.1 90) (unit 1)
     (in_bom yes) (on_board yes)
     (property "Reference" "S4" (id 0) (at 69.342 163.9316 90)
@@
     (pin "1")
   )
-  (symbol (lib_id "DL_Key_Vertical_B3F-1000:1825910-6") (at 45.72 91.44 270) (unit 1)
+  (symbol (lib_id "3rd_B3F-1000(Key_Vertical):1825910-6") (at 45.72 91.44 270) (unit 1)
     (in_bom yes) (on_board yes)
     (property "Reference" "SW1" (id 0) (at 49.53 99.06 90)
