File: Hardware/kicad_project/stm32f103.kicad_pcb (KiCad board)
At the start: 2 copper layers, 86 x 45 mm, 61 parts, among them J1 SWD, J2 USART1, J3 USB4105-GF-A, J4 Conn_01x30, J5 INA226 ALERT, J6 USB1130-15-A_REVA, M1 Mounting_Holes_3mm_THT, M2 Mounting_Holes_3mm_THT, M3 Mounting_Holes_3mm_THT, M4 Mounting_Holes_3mm_THT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

Commit message: 更新封装库
Parts:
- J3: footprint 3rd_USB4105-GF-A:3rd_USB4105-GF-A(USB-C) -> 3rd_Connector_USB:USB-C-SMD_16P_USB4105-GF-A
- J6: footprint 3rd_USB1130-15-A_REVA:3rd_USB1130-15-A_REVA(USB-A) -> 3rd_Connector_USB:USB-A-TH_4P_USB1130-15-A-REVA
- S1, S2, S3, S4: footprint 3rd_B3F-3100:3rd_B3F-3100(Key_Hori) -> 3rd_Button_Switch_THT:KEY-TH_L6.0-W6.0-H_B3F-3100
- SW1: footprint 3rd_B3F-1000:3rd_B3F-1000(Key_Vertical) -> 3rd_Button_Switch_THT:KEY-TH_L6.0-W6.0-V_B3F-1000
- U3: footprint 3rd_INA226AIDGSR:3rd_SOP50P490X110-10N(INA226AIDGSR) -> 3rd_Sensor_Power:VSSOP-10_L2.9-W5.05-P0.5_INA226AIDGSR
- U4: footprint 3rd_W25Q32JVSSIQ:3rd_SOIC127P790X216-8N(W25Q32JVSSIQ) -> 3rd_Memory_Flash:SOIC-8_L4.8-W5.8-P1.27_W25Q32JVSS
