File: Hardware/kicad_project/stm32f103.kicad_sch (KiCad schematic)
At the start: 57 parts, among them J1 SWD, J2 USART1, J3 USB4105-GF-A, J4 Conn_01x30, J5 INA226 ALERT, J6 USB1130-15-A_REVA, Q1 Q_PNP_BEC, SW1 1825910-6, U1 LM1117-3.3, U2 STM32F103RCTx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

Commit message: 更新封装库
Parts:
- J3: footprint 3rd_USB4105-GF-A:3rd_USB4105-GF-A(USB-C) -> 3rd_Connector_USB:USB-C-SMD_16P_USB4105-GF-A
- J6: footprint 3rd_USB1130-15-A_REVA:3rd_USB1130-15-A_REVA(USB-A) -> 3rd_Connector_USB:USB-A-TH_4P_USB1130-15-A-REVA
- S1, S2, S3, S4: footprint 3rd_B3F-3100:3rd_B3F-3100(Key_Hori) -> 3rd_Button_Switch_THT:KEY-TH_L6.0-W6.0-H_B3F-3100
- SW1: footprint 3rd_B3F-1000:3rd_B3F-1000(Key_Vertical) -> 3rd_Button_Switch_THT:KEY-TH_L6.0-W6.0-V_B3F-1000
- U3: footprint 3rd_INA226AIDGSR:3rd_SOP50P490X110-10N(INA226AIDGSR) -> 3rd_Sensor_Power:VSSOP-10_L2.9-W5.05-P0.5_INA226AIDGSR
- U4: footprint 3rd_W25Q32JVSSIQ:3rd_SOIC127P790X216-8N(W25Q32JVSSIQ) -> 3rd_Memory_Flash:SOIC-8_L4.8-W5.8-P1.27_W25Q32JVSS
Changed lines of the file:
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@@
     (property "Reference" "U4" (id 0) (at 113.03 151.13 0))
     (property "Value" "W25Q32JVSS" (id 1) (at 128.27 151.13 0))
-    (property "Footprint" "3rd_W25Q32JVSSIQ:3rd_SOIC127P790X216-8N(W25Q32JVSSIQ)" (id 2) (at 120.65 160.02 0)
+    (property "Footprint" "3rd_Memory_Flash:SOIC-8_L4.8-W5.8-P1.27_W25Q32JVSS" (id 2) (at 120.65 160.02 0)
       (effects (font (size 1.27 1.27)) hide)
     )
@@
     (property "Reference" "U3" (id 0) (at 243.84 16.002 0))
     (property "Value" "INA226AIDGSR" (id 1) (at 243.84 18.3134 0))
-    (property "Footprint" "3rd_INA226AIDGSR:3rd_SOP50P490X110-10N(INA226AIDGSR)" (id 2) (at 243.84 38.1 0)
+    (property "Footprint" "3rd_Sensor_Power:VSSOP-10_L2.9-W5.05-P0.5_INA226AIDGSR" (id 2) (at 243.84 38.1 0)
       (effects (font (size 1.27 1.27)) (justify left bottom) hide)
     )
@@
     (property "Reference" "J3" (id 0) (at 243.84 64.3382 0))
     (property "Value" "USB4105-GF-A" (id 1) (at 243.84 66.6496 0))
-    (property "Footprint" "3rd_USB4105-GF-A:3rd_USB4105-GF-A(USB-C)" (id 2) (at 243.84 81.28 0)
+    (property "Footprint" "3rd_Connector_USB:USB-C-SMD_16P_USB4105-GF-A" (id 2) (at 243.84 81.28 0)
       (effects (font (size 1.27 1.27)) (justify left bottom) hide)
     )
@@
       (effects (font (size 1.27 1.27)) (justify right))
     )
-    (property "Footprint" "3rd_USB1130-15-A_REVA:3rd_USB1130-15-A_REVA(USB-A)" (id 2) (at 246.38 127 0)
+    (property "Footprint" "3rd_Connector_USB:USB-A-TH_4P_USB1130-15-A-REVA" (id 2) (at 246.38 127 0)
       (effects (font (size 1.27 1.27)) (justify left bottom) hide)
     )
@@
       (effects (font (size 1.27 1.27)) (justify right))
     )
-    (property "Footprint" "3rd_B3F-3100:3rd_B3F-3100(Key_Hori)" (id 2) (at 20.32 165.1 0)
+    (property "Footprint" "3rd_Button_Switch_THT:KEY-TH_L6.0-W6.0-H_B3F-3100" (id 2) (at 20.32 165.1 0)
       (effects (font (size 1.27 1.27)) (justify left bottom) hide)
     )
@@
       (effects (font (size 1.27 1.27)) (justify right))
     )
-    (property "Footprint" "3rd_B3F-3100:3rd_B3F-3100(Key_Hori)" (id 2) (at 35.56 165.1 0)
+    (property "Footprint" "3rd_Button_Switch_THT:KEY-TH_L6.0-W6.0-H_B3F-3100" (id 2) (at 35.56 165.1 0)
       (effects (font (size 1.27 1.27)) (justify left bottom) hide)
     )
@@
       (effects (font (size 1.27 1.27)) (justify right))
     )
-    (property "Footprint" "3rd_B3F-3100:3rd_B3F-3100(Key_Hori)" (id 2) (at 49.53 165.1 0)
+    (property "Footprint" "3rd_Button_Switch_THT:KEY-TH_L6.0-W6.0-H_B3F-3100" (id 2) (at 49.53 165.1 0)
       (effects (font (size 1.27 1.27)) (justify left bottom) hide)
     )
@@
       (effects (font (size 1.27 1.27)) (justify right))
     )
-    (property "Footprint" "3rd_B3F-3100:3rd_B3F-3100(Key_Hori)" (id 2) (at 63.5 165.1 0)
+    (property "Footprint" "3rd_Button_Switch_THT:KEY-TH_L6.0-W6.0-H_B3F-3100" (id 2) (at 63.5 165.1 0)
       (effects (font (size 1.27 1.27)) (justify left bottom) hide)
     )
@@
       (effects (font (size 1.27 1.27)) (justify left))
     )
-    (property "Footprint" "3rd_B3F-1000:3rd_B3F-1000(Key_Vertical)" (id 2) (at 45.72 91.44 0)
+    (property "Footprint" "3rd_Button_Switch_THT:KEY-TH_L6.0-W6.0-V_B3F-1000" (id 2) (at 45.72 91.44 0)
       (effects (font (size 1.27 1.27)) (justify left bottom) hide)
     )
@@
     )
     (path "/00000000-0000-0000-0000-00006288cde2"
-      (reference "J3") (unit 1) (value "USB4105-GF-A") (footprint "3rd_USB4105-GF-A:3rd_USB4105-GF-A(USB-C)")
+      (reference "J3") (unit 1) (value "USB4105-GF-A") (footprint "3rd_Connector_USB:USB-C-SMD_16P_USB4105-GF-A")
     )
     (path "/00000000-0000-0000-0000-0000628bf0f6"
@@
     )
     (path "/00000000-0000-0000-0000-000062890fba"
-      (reference "J6") (unit 1) (value "USB1130-15-A_REVA") (footprint "3rd_USB1130-15-A_REVA:3rd_USB1130-15-A_REVA(USB-A)")
+      (reference "J6") (unit 1) (value "USB1130-15-A_REVA") (footprint "3rd_Connector_USB:USB-A-TH_4P_USB1130-15-A-REVA")
     )
     (path "/00000000-0000-0000-0000-000062b107ba"
@@
     )
     (path "/00000000-0000-0000-0000-000062893c59"
-      (reference "S1") (unit 1) (value "1-1825027-1") (footprint "3rd_B3F-3100:3rd_B3F-3100(Key_Hori)")
+      (reference "S1") (unit 1) (value "1-1825027-1") (footprint "3rd_Button_Switch_THT:KEY-TH_L6.0-W6.0-H_B3F-3100")
     )
     (path "/00000000-0000-0000-0000-000062894d52"
-      (reference "S2") (unit 1) (value "1-1825027-1") (footprint "3rd_B3F-3100:3rd_B3F-3100(Key_Hori)")
+      (reference "S2") (unit 1) (value "1-1825027-1") (footprint "3rd_Button_Switch_THT:KEY-TH_L6.0-W6.0-H_B3F-3100")
     )
     (path "/00000000-0000-0000-0000-0000628953c7"
-      (reference "S3") (unit 1) (value "1-1825027-1") (footprint "3rd_B3F-3100:3rd_B3F-3100(Key_Hori)")
+      (reference "S3") (unit 1) (value "1-1825027-1") (footprint "3rd_Button_Switch_THT:KEY-TH_L6.0-W6.0-H_B3F-3100")
     )
     (path "/00000000-0000-0000-0000-000062895c6f"
-      (reference "S4") (unit 1) (value "1-1825027-1") (footprint "3rd_B3F-3100:3rd_B3F-3100(Key_Hori)")
+      (reference "S4") (unit 1) (value "1-1825027-1") (footprint "3rd_Button_Switch_THT:KEY-TH_L6.0-W6.0-H_B3F-3100")
     )
     (path "/00000000-0000-0000-0000-0000628b7f60"
-      (reference "SW1") (unit 1) (value "1825910-6") (footprint "3rd_B3F-1000:3rd_B3F-1000(Key_Vertical)")
+      (reference "SW1") (unit 1) (value "1825910-6") (footprint "3rd_Button_Switch_THT:KEY-TH_L6.0-W6.0-V_B3F-1000")
     )
     (path "/00000000-0000-0000-0000-00006249904c"
@@
     )
     (path "/00000000-0000-0000-0000-0000628758b5"
-      (reference "U3") (unit 1) (value "INA226AIDGSR") (footprint "3rd_INA226AIDGSR:3rd_SOP50P490X110-10N(INA226AIDGSR)")
+      (reference "U3") (unit 1) (value "INA226AIDGSR") (footprint "3rd_Sensor_Power:VSSOP-10_L2.9-W5.05-P0.5_INA226AIDGSR")
     )
     (path "/00000000-0000-0000-0000-0000626c79c4"
-      (reference "U4") (unit 1) (value "W25Q32JVSS") (footprint "3rd_W25Q32JVSSIQ:3rd_SOIC127P790X216-8N(W25Q32JVSSIQ)")
+      (reference "U4") (unit 1) (value "W25Q32JVSS") (footprint "3rd_Memory_Flash:SOIC-8_L4.8-W5.8-P1.27_W25Q32JVSS")
     )
     (path "/00000000-0000-0000-0000-000062486c0f"
